Commit message: 奖励函数设计完成

File: source/ur5e/ur5e/tasks/manager_based/usd/ur5e_zhiyuan/urdf/ur5e.urdf (robot description, URDF)
Before this commit: robot ur5e, 36 links, 35 joints
Joints:
- joint catch_joint: origin xyz=-0.035 0.28 0.05 rpy=-1.5708 -1.5708 0.0 -> xyz=-0.035 0.25 0.05 rpy=0.0 0.0 0.0
- joint elbow_joint: limit lower=-3.14159265359 upper=3.14159265359 effort=150.0 velocity=3.14 -> lower=-2.0 upper=2.0 effort=150.0 velocity=3.14
- joint shoulder_lift_joint: limit lower=-6.28318530718 upper=6.28318530718 effort=150.0 velocity=3.14 -> lower=-3.14 upper=3.14 effort=150.0 velocity=3.14
- joint wrist_1_joint: limit lower=-6.28318530718 upper=6.28318530718 effort=28.0 velocity=6.28 -> lower=-3.14159 upper=3.14159 effort=28.0 velocity=6.28
- joint wrist_2_joint: limit lower=-6.28318530718 upper=6.28318530718 effort=28.0 velocity=6.28 -> lower=-2.0 upper=2.0 effort=28.0 velocity=6.28
- joint wrist_3_joint: limit lower=-6.28318530718 upper=6.28318530718 effort=28.0 velocity=6.28 -> lower=-3.14159 upper=0 effort=28.0 velocity=6.28

Commit message: 单指抓取

File: source/ur5e/ur5e/tasks/manager_based/usd/ur5e_zhiyuan/urdf/ur5e.urdf (robot description, URDF)
Before this commit: robot ur5e, 36 links, 35 joints
Joints:
- joint l_f_joint2_1: type revolute -> fixed
- joint l_f_joint3_1: type revolute -> fixed
- joint l_f_joint3_2: type revolute -> fixed
- joint l_f_joint3_3: type revolute -> fixed

Commit message: 能抓起的奖励函数

File: source/ur5e/ur5e/tasks/manager_based/usd/ur5e_zhiyuan/urdf/ur5e.urdf (robot description, URDF)
Before this commit: robot ur5e, 36 links, 35 joints
Joints:
- joint catch_joint: origin xyz=-0.035 0.25 0.05 rpy=0.0 0.0 0.0 -> xyz=-0.015 0.22 0.05 rpy=0.0 0.0 0.0
